File: pcb_design/Light Board/TR109-lightboard.kicad_pcb (KiCad board)
At the start: 2 copper layers, 49 x 18 mm, 11 parts, among them J1 Conn_01x05_Female

Commit message: Pcb and shell design work
Parts:
- added REF**: MountingHole_2.1mm, MountingHole:MountingHole_2.1mm, F.Cu at (169.0, 108.6)
- added REF**: MountingHole_2.1mm, MountingHole:MountingHole_2.1mm, F.Cu at (127.0, 94.8)
- moved R4 5.72 mm to (165.2, 105.3), turned to 180 degrees
Routing:
- net Net-(D4-Pad1): track 10.4 -> 14.0 mm
Other:
- board size 49 x 18 mm -> 49.7 x 18.2 mm
Changed lines of the file:
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@@
   (general
     (thickness 1.6)
-    (drawings 24)
-    (tracks 27)
+    (drawings 8)
+    (tracks 29)
     (zones 0)
-    (modules 11)
+    (modules 13)
     (nets 10)
   )
@@
     (add_net "Net-(D4-Pad1)")
   )
+  (module MountingHole:MountingHole_2.1mm (layer F.Cu)
+    (at 169.03 108.57)
+    (descr "Mounting Hole 2.1mm, no annular")
+    (tags "mounting hole 2.1mm no annular")
+    (attr virtual)
+    (fp_text reference REF** (at 0 -3.2) (layer F.Fab)
+      (effects (font (size 1 1) (thickness 0.15)))
+    )
+    (fp_text value MountingHole_2.1mm (at 0 3.2) (layer F.Fab)
+      (effects (font (size 1 1) (thickness 0.15)))
+    )
+    (fp_text user %R (at 0.3 0) (layer F.Fab)
+      (effects (font (size 1 1) (thickness 0.15)))
+    )
+    (fp_circle (center 0 0) (end 2.1 0) (layer Cmts.User) (width 0.15))
+    (fp_circle (center 0 0) (end 2.35 0) (layer F.CrtYd) (width 0.05))
+    (pad "" np_thru_hole circle (at 0 0) (size 2.1 2.1) (drill 2.1) (layers *.Cu *.Mask))
+  )
+  (module MountingHole:MountingHole_2.1mm (layer F.Cu)
+    (at 127.04 94.78)
+    (descr "Mounting Hole 2.1mm, no annular")
+    (tags "mounting hole 2.1mm no annular")
+    (attr virtual)
+    (fp_text reference REF** (at 0 -3.2) (layer F.Fab)
+      (effects (font (size 1 1) (thickness 0.15)))
+    )
+    (fp_text value MountingHole_2.1mm (at 0 3.2) (layer F.Fab)
+      (effects (font (size 1 1) (thickness 0.15)))
+    )
+    (fp_text user %R (at 0.3 0) (layer F.Fab)
+      (effects (font (size 1 1) (thickness 0.15)))
+    )
+    (fp_circle (center 0 0) (end 2.1 0) (layer Cmts.User) (width 0.15))
+    (fp_circle (center 0 0) (end 2.35 0) (layer F.CrtYd) (width 0.05))
+    (pad "" np_thru_hole circle (at 0 0) (size 2.1 2.1) (drill 2.1) (layers *.Cu *.Mask))
+  )
   (module Connector_PinHeader_2.00mm:PinHeader_1x05_P2.00mm_Vertical (layer F.Cu)
     (at 145.396704 95.3135 90)
@@
     )
     (fp_text value Conn_01x05_Female (at 0 10.06 90) (layer F.Fab)
-      (effects (font (size 1 1) (thickness 0.15)))
-    )
-    (fp_text user %R (at 0 4) (layer F.Fab)
       (effects (font (size 1 1) (thickness 0.15)))
     )
@@
     (fp_line (start 1.5 9.5) (end 1.5 -1.5) (layer F.CrtYd) (width 0.05))
     (fp_line (start 1.5 -1.5) (end -1.5 -1.5) (layer F.CrtYd) (width 0.05))
+    (fp_text user %R (at 0 4) (layer F.Fab)
+      (effects (font (size 1 1) (thickness 0.15)))
+    )
     (pad 5 thru_hole oval (at 0 8 90) (size 1.35 1.35) (drill 0.8) (layers *.Cu *.Mask)
       (net 5 L1))
@@
   )
   (module Resistor_SMD:R_0603_1608Metric_Pad0.98x0.95mm_HandSolder (layer F.Cu)
-    (at 170.7375 106.5784 270)
+    (at 165.16 105.3 180)
     (descr "Resistor SMD 0603 (1608 Metric), square (rectangular) end terminal, IPC_7351 nominal with elongated pad for handsoldering. (Body size source: IPC-SM-782 page 72, https://www.pcb-3d.com/wordpress/wp-content/uploads/ipc-sm-782a_amendment_1_and_2.pdf), generated with kicad-footprint-generator")
     (tags "resistor handsolder")
     (attr smd)
-    (fp_text reference R4 (at 0 -1.43 90) (layer F.SilkS)
-      (effects (font (size 1 1) (thickness 0.15)))
-    )
-    (fp_text value R (at 0 1.43 90) (layer F.Fab)
+    (fp_text reference R4 (at 0 -1.43) (layer F.SilkS)
+      (effects (font (size 1 1) (thickness 0.15)))
+    )
+    (fp_text value R (at 0 1.43) (layer F.Fab)
       (effects (font (size 1 1) (thickness 0.15)))
     )
@@
     (fp_line (start -0.8 -0.4125) (end 0.8 -0.4125) (layer F.Fab) (width 0.1))
     (fp_line (start -0.8 0.4125) (end -0.8 -0.4125) (layer F.Fab) (width 0.1))
-    (fp_text user %R (at 0 0 90) (layer F.Fab)
-      (effects (font (size 0.4 0.4) (thickness 0.06)))
-    )
-    (pad 2 smd roundrect (at 0.9125 0 270) (size 0.975 0.95) (layers F.Cu F.Paste F.Mask) (roundrect_rratio 0.25)
+    (fp_text user %R (at 0 0) (layer F.Fab)
+      (effects (font (size 0.4 0.4) (thickness 0.06)))
+    )
+    (pad 2 smd roundrect (at 0.9125 0 180) (size 0.975 0.95) (layers F.Cu F.Paste F.Mask) (roundrect_rratio 0.25)
       (net 9 GND))
-    (pad 1 smd roundrect (at -0.9125 0 270) (size 0.975 0.95) (layers F.Cu F.Paste F.Mask) (roundrect_rratio 0.25)
+    (pad 1 smd roundrect (at -0.9125 0 180) (size 0.975 0.95) (layers F.Cu F.Paste F.Mask) (roundrect_rratio 0.25)
       (net 6 "Net-(D4-Pad1)"))
     (model ${KISYS3DMOD}/Resistor_SMD.3dshapes/R_0603_1608Metric.wrl
@@
     )
   )
-  (gr_line (start 124.994595 93.447305) (end 125.207622 93.029119) (layer Edge.Cuts) (width 0.2))
-  (gr_line (start 126.421172 110.457096) (end 172.372236 110.457096) (layer Edge.Cuts) (width 0.2))
-  (gr_line (start 124.921162 108.957086) (end 124.994595 109.420626) (layer Edge.Cuts) (width 0.2))
-  (gr_line (start 125.207622 109.838756) (end 125.5395 110.170636) (layer Edge.Cuts) (width 0.2))
-  (gr_line (start 125.957627 110.383656) (end 126.421172 110.457096) (layer Edge.Cuts) (width 0.2))
-  (gr_line (start 125.207622 93.029119) (end 125.5395 92.6973) (layer Edge.Cuts) (width 0.2))
-  (gr_line (start 173.872246 108.957086) (end 173.872246 93.910791) (layer Edge.Cuts) (width 0.2))
-  (gr_line (start 125.5395 110.170636) (end 125.957627 110.383656) (layer Edge.Cuts) (width 0.2))
-  (gr_line (start 124.921162 93.910791) (end 124.921162 108.957086) (layer Edge.Cuts) (width 0.2))
-  (gr_line (start 172.372236 92.41078) (end 126.421172 92.41078) (layer Edge.Cuts) (width 0.2))
-  (gr_line (start 125.957627 92.484213) (end 126.421172 92.41078) (layer Edge.Cuts) (width 0.2))
-  (gr_line (start 173.798816 93.447246) (end 173.872246 93.910791) (layer Edge.Cuts) (width 0.2))
-  (gr_line (start 124.921162 93.910791) (end 124.994595 93.447305) (layer Edge.Cuts) (width 0.2))
-  (gr_line (start 173.872246 108.957086) (end 173.798816 109.420626) (layer Edge.Cuts) (width 0.2))
-  (gr_line (start 173.798816 109.420626) (end 173.585786 109.838756) (layer Edge.Cuts) (width 0.2))
-  (gr_line (start 173.585786 109.838756) (end 173.253906 110.170636) (layer Edge.Cuts) (width 0.2))
-  (gr_line (start 173.253906 110.170636) (end 172.835776 110.383656) (layer Edge.Cuts) (width 0.2))
-  (gr_line (start 172.835776 110.383656) (end 172.372236 110.457096) (layer Edge.Cuts) (width 0.2))
-  (gr_line (start 172.372236 92.41078) (end 172.835776 92.484213) (layer Edge.Cuts) (width 0.2))
-  (gr_line (start 172.835776 92.484213) (end 173.253906 92.6973) (layer Edge.Cuts) (width 0.2))
-  (gr_line (start 173.253906 92.6973) (end 173.585786 93.029119) (layer Edge.Cuts) (width 0.2))
-  (gr_line (start 173.585786 93.029119) (end 173.798816 93.447246) (layer Edge.Cuts) (width 0.2))
-  (gr_line (start 124.994595 109.420626) (end 125.207622 109.838756) (layer Edge.Cuts) (width 0.2))
-  (gr_line (start 125.5395 92.6973) (end 125.957627 92.484213) (layer Edge.Cuts) (width 0.2))
+  (gr_arc (start 172.503408 108.9935) (end 172.581352 110.571454) (angle -90) (layer Edge.Cuts) (width 0.2))
+  (gr_arc (start 126.000359 108.956197) (end 124.385101 109.071444) (angle -81.8377804) (layer Edge.Cuts) (width 0.2))
+  (gr_arc (start 125.943267 93.939003) (end 125.885111 92.380837) (angle -89.9999618) (layer Edge.Cuts) (width 0.2))
+  (gr_arc (start 172.488819 93.973381) (end 174.081362 93.880848) (angle -83.34927126) (layer Edge.Cuts) (width 0.2))
+  (gr_line (start 172.581352 92.380837) (end 125.885111 92.380837) (layer Edge.Cuts) (width 0.2))
+  (gr_line (start 124.385101 93.997158) (end 124.385101 109.071444) (layer Edge.Cuts) (width 0.2))
+  (gr_line (start 174.081362 108.915555) (end 174.081362 93.880848) (layer Edge.Cuts) (width 0.2))
+  (gr_line (start 125.885111 110.571454) (end 172.581352 110.571454) (layer Edge.Cuts) (width 0.2))
   (segment (start 148.412 100) (end 156.6661 100) (width 0.127) (layer F.Cu) (net 1))
   (segment (start 156.6661 100) (end 158.9138 102.2477) (width 0.127) (layer F.Cu) (net 1))
@@
   (segment (start 170.7375 95.3135) (end 170.7375 99.0219) (width 0.127) (layer F.Cu) (net 6))
   (segment (start 170.7375 99.0219) (end 170.7375 102.7176) (width 0.127) (layer F.Cu) (net 6))
-  (segment (start 170.7375 102.7176) (end 170.7375 105.6659) (width 0.127) (layer F.Cu) (net 6))
+  (segment (start 166.0725 105.3) (end 169.6 105.3) (width 0.127) (layer F.Cu) (net 6))
+  (segment (start 170.7375 104.1625) (end 170.7375 102.7176) (width 0.127) (layer F.Cu) (net 6))
+  (segment (start 169.6 105.3) (end 170.7375 104.1625) (width 0.127) (layer F.Cu) (net 6))
   (segment (start 151.396704 95.3135) (end 152.603204 96.52) (width 0.127) (layer F.Cu) (net 7))
   (segment (start 152.603204 96.52) (end 168.0464 96.52) (width 0.127) (layer F.Cu) (net 7))

Commit message: Rev 3 board changes, blender file changes
Other:
- rule pad_to_mask_clearance: 0.2 -> 0

Commit message: Pcb and enclosure changes for proto 01
Parts:
- D1, D2, D3, D4, D5, D6: footprint LED_SMD:LED_0603_1608Metric_Pad1.05x0.95mm_HandSolder -> LED_SMD:LED_1206_3216Metric_Pad1.42x1.75mm_HandSolder

Commit message: parts changes
Parts:
- R1, R2, R3, R4: footprint Resistor_SMD:R_0603_1608Metric_Pad0.98x0.95mm_HandSolder -> Resistor_SMD:R_0805_2012Metric_Pad1.20x1.40mm_HandSolder
- moved R1 5.13 mm to (131.6, 106.5), turned to 90 degrees
- moved R2 5.05 mm to (144.1, 106.5), turned to 90 degrees
- moved R3 4.96 mm to (156.6, 106.5), turned to 90 degrees
Routing:
- net Net-(D3-Pad1): track 2.25 -> 3.25 mm
- net Net-(D2-Pad1): track 2.37 -> 3.29 mm
- net Net-(D1-Pad1): track 2.60 -> 3.23 mm
