File: pcb_design/Light Board/TR109-lightboard.sch (KiCad schematic (older format))
At the start: 11 parts, among them J1 Conn_01x05_Female

Commit message: Pcb and enclosure changes for proto 01
Parts:
- D1, D2, D3, D4, D5, D6: footprint LED_SMD:LED_0603_1608Metric_Pad1.05x0.95mm_HandSolder -> LED_SMD:LED_1206_3216Metric_Pad1.42x1.75mm_HandSolder
Changed lines of the file:
@@
 F 0 "D1" H 4893 4567 50  0000 C CNN
 F 1 "LED" H 4893 4476 50  0000 C CNN
-F 2 "LED_SMD:LED_0603_1608Metric_Pad1.05x0.95mm_HandSolder" H 4900 4350 50  0001 C CNN
+F 2 "LED_SMD:LED_1206_3216Metric_Pad1.42x1.75mm_HandSolder" H 4900 4350 50  0001 C CNN
 F 3 "~" H 4900 4350 50  0001 C CNN
 	1    4900 4350
@@
 F 0 "D2" H 5693 4567 50  0000 C CNN
 F 1 "LED" H 5693 4476 50  0000 C CNN
-F 2 "LED_SMD:LED_0603_1608Metric_Pad1.05x0.95mm_HandSolder" H 5700 4350 50  0001 C CNN
+F 2 "LED_SMD:LED_1206_3216Metric_Pad1.42x1.75mm_HandSolder" H 5700 4350 50  0001 C CNN
 F 3 "~" H 5700 4350 50  0001 C CNN
 	1    5700 4350
@@
 F 0 "D3" H 6493 4567 50  0000 C CNN
 F 1 "LED" H 6493 4476 50  0000 C CNN
-F 2 "LED_SMD:LED_0603_1608Metric_Pad1.05x0.95mm_HandSolder" H 6500 4350 50  0001 C CNN
+F 2 "LED_SMD:LED_1206_3216Metric_Pad1.42x1.75mm_HandSolder" H 6500 4350 50  0001 C CNN
 F 3 "~" H 6500 4350 50  0001 C CNN
 	1    6500 4350
@@
 F 0 "D4" H 8493 4317 50  0000 C CNN
 F 1 "LED" H 8493 4226 50  0000 C CNN
-F 2 "LED_SMD:LED_0603_1608Metric_Pad1.05x0.95mm_HandSolder" H 8500 4100 50  0001 C CNN
+F 2 "LED_SMD:LED_1206_3216Metric_Pad1.42x1.75mm_HandSolder" H 8500 4100 50  0001 C CNN
 F 3 "~" H 8500 4100 50  0001 C CNN
 	1    8500 4100
@@
 F 0 "D5" H 8493 4867 50  0000 C CNN
 F 1 "LED" H 8493 4776 50  0000 C CNN
-F 2 "LED_SMD:LED_0603_1608Metric_Pad1.05x0.95mm_HandSolder" H 8500 4650 50  0001 C CNN
+F 2 "LED_SMD:LED_1206_3216Metric_Pad1.42x1.75mm_HandSolder" H 8500 4650 50  0001 C CNN
 F 3 "~" H 8500 4650 50  0001 C CNN
 	1    8500 4650
@@
 F 0 "D6" H 8493 5467 50  0000 C CNN
 F 1 "LED" H 8493 5376 50  0000 C CNN
-F 2 "LED_SMD:LED_0603_1608Metric_Pad1.05x0.95mm_HandSolder" H 8500 5250 50  0001 C CNN
+F 2 "LED_SMD:LED_1206_3216Metric_Pad1.42x1.75mm_HandSolder" H 8500 5250 50  0001 C CNN
 F 3 "~" H 8500 5250 50  0001 C CNN
 	1    8500 5250

Commit message: parts changes
Parts:
- R1, R2, R3, R4: footprint Resistor_SMD:R_0603_1608Metric_Pad0.98x0.95mm_HandSolder -> Resistor_SMD:R_0805_2012Metric_Pad1.20x1.40mm_HandSolder
Changed lines of the file:
@@
 F 0 "R4" V 7693 4650 50  0000 C CNN
 F 1 "R" V 7784 4650 50  0000 C CNN
-F 2 "Resistor_SMD:R_0603_1608Metric_Pad0.98x0.95mm_HandSolder" V 7830 4650 50  0001 C CNN
+F 2 "Resistor_SMD:R_0805_2012Metric_Pad1.20x1.40mm_HandSolder" V 7830 4650 50  0001 C CNN
 F 3 "~" H 7900 4650 50  0001 C CNN
 	1    7900 4650
@@
 F 0 "R3" H 6080 4804 50  0000 R CNN
 F 1 "R" H 6080 4895 50  0000 R CNN
-F 2 "Resistor_SMD:R_0603_1608Metric_Pad0.98x0.95mm_HandSolder" V 6080 4850 50  0001 C CNN
+F 2 "Resistor_SMD:R_0805_2012Metric_Pad1.20x1.40mm_HandSolder" V 6080 4850 50  0001 C CNN
 F 3 "~" H 6150 4850 50  0001 C CNN
 	1    6150 4850
@@
 F 0 "R2" H 5230 4804 50  0000 R CNN
 F 1 "R" H 5230 4895 50  0000 R CNN
-F 2 "Resistor_SMD:R_0603_1608Metric_Pad0.98x0.95mm_HandSolder" V 5230 4850 50  0001 C CNN
+F 2 "Resistor_SMD:R_0805_2012Metric_Pad1.20x1.40mm_HandSolder" V 5230 4850 50  0001 C CNN
 F 3 "~" H 5300 4850 50  0001 C CNN
 	1    5300 4850
@@
 F 0 "R1" H 4480 4804 50  0000 R CNN
 F 1 "R" H 4480 4895 50  0000 R CNN
-F 2 "Resistor_SMD:R_0603_1608Metric_Pad0.98x0.95mm_HandSolder" V 4480 4850 50  0001 C CNN
+F 2 "Resistor_SMD:R_0805_2012Metric_Pad1.20x1.40mm_HandSolder" V 4480 4850 50  0001 C CNN
 F 3 "~" H 4550 4850 50  0001 C CNN
 	1    4550 4850
