File: pcb_design/Sensor Board/tr109-sensorboard.kicad_pcb (KiCad board)
At the start: 2 copper layers, 65 x 30 mm, 57 parts, among them J1 Conn_01x01_Female, J2 Conn_01x01_Female, J3 Conn_01x04_Female, J47 Raspberry_Pi_2_3, U1 BME680, U2 74HC595, U3 AMG8833

Commit message: kicad v8
Parts:
- D1, D10, D2, D3, D4, D5, D6, D7, D8, D9: value G-LED -> Green_LED
- D11, D12: value R-LED -> Red_LED
- D13, D14, D17, D18: value B-LED -> Blue_LED
- D15, D16: value Y-LED -> Yellow_LED
Connections:
- J47 pad 10: Net-(J47-Pad10) -> unconnected-(J47-GPIO15/RXD-Pad10)
- J47 pad 11: Net-(J47-Pad11) -> unconnected-(J47-GPIO17-Pad11)
- J47 pad 12: Net-(J47-Pad12) -> unconnected-(J47-GPIO18/PWM0-Pad12)
- J47 pad 13: Net-(J47-Pad13) -> unconnected-(J47-GPIO27-Pad13)
- J47 pad 15: Net-(J47-Pad15) -> unconnected-(J47-GPIO22-Pad15)
- J47 pad 16: Net-(J47-Pad16) -> unconnected-(J47-GPIO23-Pad16)
- J47 pad 18: Net-(J47-Pad18) -> unconnected-(J47-GPIO24-Pad18)
- J47 pad 19: Net-(J47-Pad19) -> unconnected-(J47-MOSI0/GPIO10-Pad19)
- J47 pad 21: Net-(J47-Pad21) -> unconnected-(J47-MISO0/GPIO9-Pad21)
- J47 pad 22: Net-(J47-Pad22) -> unconnected-(J47-GPIO25-Pad22)
- J47 pad 23: Net-(J47-Pad23) -> unconnected-(J47-SCLK0/GPIO11-Pad23)
- J47 pad 24: Net-(J47-Pad24) -> unconnected-(J47-~{CE0}/GPIO8-Pad24)
- J47 pad 26: Net-(J47-Pad26) -> unconnected-(J47-~{CE1}/GPIO7-Pad26)
- J47 pad 27: Net-(J47-Pad27) -> unconnected-(J47-ID_SD/GPIO0-Pad27)
- J47 pad 28: Net-(J47-Pad28) -> unconnected-(J47-ID_SC/GPIO1-Pad28)
- J47 pad 29: Net-(J47-Pad29) -> unconnected-(J47-GCLK1/GPIO5-Pad29)
- J47 pad 31: Net-(J47-Pad31) -> unconnected-(J47-GCLK2/GPIO6-Pad31)
- J47 pad 32: Net-(J47-Pad32) -> unconnected-(J47-PWM0/GPIO12-Pad32)
- J47 pad 33: Net-(J47-Pad33) -> unconnected-(J47-PWM1/GPIO13-Pad33)
- J47 pad 36: Net-(J47-Pad36) -> unconnected-(J47-GPIO16-Pad36)
- J47 pad 38: Net-(J47-Pad38) -> unconnected-(J47-GPIO20/MOSI1-Pad38)
- J47 pad 7: Net-(J47-Pad7) -> unconnected-(J47-GCLK0/GPIO4-Pad7)
- J47 pad 8: Net-(J47-Pad8) -> unconnected-(J47-GPIO14/TXD-Pad8)
- U2 pad 6: Net-(U2-Pad6) -> unconnected-(U2-QG-Pad6)
- U2 pad 9: Net-(U2-Pad9) -> unconnected-(U2-QH'-Pad9)
- U3 pad 1: Net-(U3-Pad1) -> unconnected-(U3-NC-Pad1)
- U3 pad 11: Net-(U3-Pad11) -> unconnected-(U3-NC-Pad11)
- U3 pad 14: Net-(U3-Pad14) -> unconnected-(U3-NC-Pad14)
- U3 pad 7: Net-(U3-Pad7) -> unconnected-(U3-NC-Pad7)
- U3 pad 8: Net-(U3-Pad8) -> unconnected-(U3-NC-Pad8)
Routing:
- net unconnected-(J47-GPIO22-Pad15): track 0.00 -> 1.51 mm
- net Net-(J47-Pad15): track 1.51 -> 0.00 mm
Other:
- net class Default removed
- board text added: "TBH/VOC/EXP/TC - REV 4"
- board text removed: "TBH/VOC/EXP/TC - REV 3"
